Commit message: puppypi_description: add fixed_legs xacro argument
fixed_legs:=true makes all 8 leg joints fixed and locks joint1 at
0.8 rad, the standing pose from the ROS 1 puppy_sim spawn arguments.
A fixed joint has no angle, so the 0.8 is added to the joint origin's
roll instead; joint1 rotates about x, so the two rotations add.
Gazebo then merges the robot into one rigid body that stands and can
be moved as a whole.

The default is false, which produces the same URDF as before, so the
real robot and robot_description.launch.py are unaffected.

File: src/simulations/puppypi_description/urdf/puppy.xacro (robot description, xacro)
@@ -6,4 +6,14 @@
   <xacro:property name="motor_torque" value="0.5"/>
   <xacro:property name="motor_vec" value="2"/>
+  <!-- fixed_legs=true locks all 8 leg joints in a standing pose for the Gazebo sim -->
+  <xacro:arg name="fixed_legs" default="false"/>
+  <xacro:if value="$(arg fixed_legs)">
+    <xacro:property name="leg_joint_type" value="fixed"/>
+    <xacro:property name="stand_joint1" value="0.8"/>
+  </xacro:if>
+  <xacro:unless value="$(arg fixed_legs)">
+    <xacro:property name="leg_joint_type" value="revolute"/>
+    <xacro:property name="stand_joint1" value="0.0"/>
+  </xacro:unless>
   <link name="base_footprint" />
   <joint name="base_joint" type="fixed">
@@ -127,8 +137,8 @@
   <joint
     name="lb_joint1"
-    type="revolute">
+    type="${leg_joint_type}">
     <origin
       xyz="0.0420105649539 0.0778693100523862 0.0159880060021007"
-      rpy="-0.752 0 0" />
+      rpy="${-0.752 + stand_joint1} 0 0" />
     <parent
       link="base_dummy" />
@@ -183,5 +193,5 @@
   <joint
     name="lb_joint2"
-    type="revolute">
+    type="${leg_joint_type}">
     <origin
       xyz="0.0120498902789596 0.0525235728370777 -0.052877465200695"
@@ -239,8 +249,8 @@
   <joint
     name="rb_joint1"
-    type="revolute">
+    type="${leg_joint_type}">
     <origin
       xyz="-0.0420105649534512 0.0778693100523859 0.0159880060091649"
-      rpy="-0.752 0 0" />
+      rpy="${-0.752 + stand_joint1} 0 0" />
     <parent
       link="base_dummy" />
@@ -295,5 +305,5 @@
   <joint
     name="rb_joint2"
-    type="revolute">
+    type="${leg_joint_type}">
     <origin
       xyz="-0.0185498902789654 0.0525235728370851 -0.0528774652006949"
@@ -351,8 +361,8 @@
   <joint
     name="rf_joint1"
-    type="revolute">
+    type="${leg_joint_type}">
     <origin
       xyz="-0.0420105469986279 -0.0778692767711234 0.0106512951143373"
-      rpy="-0.752 0 0" />
+      rpy="${-0.752 + stand_joint1} 0 0" />
     <parent
       link="base_dummy" />
@@ -407,5 +417,5 @@
   <joint
     name="rf_joint2"
-    type="revolute">
+    type="${leg_joint_type}">
     <origin
       xyz="-0.0185498902789602 0.0525235728370692 -0.0528774652007036"
@@ -463,8 +473,8 @@
   <joint
     name="lf_joint1"
-    type="revolute">
+    type="${leg_joint_type}">
     <origin
       xyz="0.0420105469981795 -0.0778692767711239 0.0106512951072731"
-      rpy="-0.752 0 0" />
+      rpy="${-0.752 + stand_joint1} 0 0" />
     <parent
       link="base_dummy" />
@@ -519,5 +529,5 @@
   <joint
     name="lf_joint2"
-    type="revolute">
+    type="${leg_joint_type}">
     <origin
       xyz="0.0120498902789604 0.0525235728370695 -0.0528774652007036"
